File: carte alimentation/carte alimentation.kicad_sch (KiCad schematic)
At the start: 17 parts, among them J1 con BAT, J10 INCASE, J11 CP Dynamixel, J12 INCASE, J13 ventilo 1, J14 ventilo 2, J15 CD, J16 con BAT, J17 BAU, J2 CP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

Commit message: on commence trankil mimil
Parts:
- removed J1: con BAT, Connector_AMASS:AMASS_XT60-F_1x02_P7.20mm_Vertical, symbol Connector_Generic:Conn_01x02
- removed J15: CD, Connector_Molex:Molex_KK-254_AE-6410-02A_1x02_P2.54mm_Vertical, symbol Connector_Generic:Conn_01x02
Connections:
- net +24V: no longer J13.2 (Pin_2), J14.2 (Pin_2)
- net +5V: now also J13.2 (Pin_2), J14.2 (Pin_2)
Other:
- moved on the sheet: J10, J11, J12, J13, J14, J16, J17, J6, J7, J8, J9

Commit message: traco
Parts:
- removed J16: con BAT, Connector_AMASS:AMASS_XT60-M_1x02_P7.20mm_Vertical, symbol Connector_Generic:Conn_01x02
- removed J17: BAU, Connector_Molex:Molex_KK-396_A-41791-0002_1x02_P3.96mm_Vertical, symbol Connector_Generic:Conn_01x02
- added Batcon1: Conn_01x02, Connector_AMASS:AMASS_XT60-F_1x02_P7.20mm_Vertical, symbol Connector_Generic:Conn_01x02
- added Bau.1: Conn_01x02, Connector_Molex:Molex_KK-254_AE-6410-02A_1x02_P2.54mm_Vertical, symbol Connector_Generic:Conn_01x02
- added D1: D, Diode_THT:D_DO-35_SOD27_P10.16mm_Horizontal, symbol Device:D
- added D3, D4, D5, D6, D7: LED_Small, LED_SMD:LED_1206_3216Metric_Pad1.42x1.75mm_HandSolder, symbol Device:LED_Small
- added K1: TE_PCH-1xxx2M, Relay_THT:Relay_SPST_TE_PCH-1xxx2M, symbol Relay:TE_PCH-1xxx2M
- added PS1: TEN_50-2411, TEN_50-2411:TEN50_TRP, symbol TEN_50-2411:TEN_50-2411
- added R25, R26, R27, R28, R29: R_Small, LED_SMD:LED_1206_3216Metric_Pad1.42x1.75mm_HandSolder, symbol Device:R_Small
- added U4: TSR1-2433E, Converter_DCDC:Converter_DCDC_TRACO_TSR1-xxxxE_THT, symbol Regulator_Switching:TSR1-2433E
- added U6: TSR1-2450E, Converter_DCDC:Converter_DCDC_TRACO_TSR1-xxxxE_THT, symbol Regulator_Switching:TSR1-2450E
Connections:
- net +12V: now also R28.1
- net +24V: now also K1.2, PS1.1 (+VIN(VCC)), R25.1, U4.1 (Vin), U6.1 (Vin)
- net +5V: now also R26.1, U6.3 (Vout)
- net +BATT: now also Batcon1.2 (Pin_2), Bau.1.2 (Pin_2), K1.3, R29.1
- net GND: now also Batcon1.1 (Pin_1), D1.2 (A), D3.1 (K), D4.1 (K), D5.1 (K), D6.1 (K), D7.1 (K), K1.1, PS1.2 (-VIN(GND)), PS1.5 (-VOUT), U4.2 (GND), U6.2 (GND)
- new net: D6.2 (A), R28.2
- new net: D4.2 (A), R26.2
- new net: D5.2 (A), R27.2
- new net: D3.2 (A), R25.2
- new net: D7.2 (A), R29.2
- new net +3.3V: U4.3 (Vout)
- new net +5VP: PS1.4 (+VOUT), R27.1
- new net Bau: Bau.1.1 (Pin_1), D1.1 (K), K1.5
- no-connect marks 0 -> 2

Commit message: on avance doucement
Parts:
- removed D3, D4, D5, D6, D7: LED_Small, LED_SMD:LED_1206_3216Metric_Pad1.42x1.75mm_HandSolder, symbol Device:LED_Small
- removed J10, J12: INCASE, Connector_AMASS:AMASS_XT60-F_1x02_P7.20mm_Vertical, symbol Connector_Generic:Conn_01x02
- removed J11: CP Dynamixel, Connector_AMASS:AMASS_XT60-F_1x02_P7.20mm_Vertical, symbol Connector_Generic:Conn_01x02
- removed J13: ventilo 1, Connector_Molex:Molex_KK-254_AE-6410-02A_1x02_P2.54mm_Vertical, symbol Connector_Generic:Conn_01x02
- removed J14: ventilo 2, Connector_Molex:Molex_KK-254_AE-6410-02A_1x02_P2.54mm_Vertical, symbol Connector_Generic:Conn_01x02
- removed J2: CP, Connector_Molex:Molex_KK-254_AE-6410-02A_1x02_P2.54mm_Vertical, symbol Connector_Generic:Conn_01x02
- removed J3: CD, Connector_Molex:Molex_KK-254_AE-6410-02A_1x02_P2.54mm_Vertical, symbol Connector_Generic:Conn_01x02
- removed J4: CL, Connector_Molex:Molex_KK-254_AE-6410-02A_1x02_P2.54mm_Vertical, symbol Connector_Generic:Conn_01x02
- removed J5: CC, Connector_Molex:Molex_KK-254_AE-6410-02A_1x02_P2.54mm_Vertical, symbol Connector_Generic:Conn_01x02
- removed J6: CE, Connector_Molex:Molex_KK-254_AE-6410-02A_1x02_P2.54mm_Vertical, symbol Connector_Generic:Conn_01x02
- removed J7, J8: I2C ext, Connector_Molex:Molex_KK-254_AE-6410-02A_1x02_P2.54mm_Vertical, symbol Connector_Generic:Conn_01x02
- removed J9: CD, Connector_AMASS:AMASS_XT60-F_1x02_P7.20mm_Vertical, symbol Connector_Generic:Conn_01x02
- removed R25, R26, R27, R28, R29: R_Small, LED_SMD:LED_1206_3216Metric_Pad1.42x1.75mm_HandSolder, symbol Device:R_Small
- added PS2: TEN_50-2411, TEN_50-2411:TEN50_TRP, symbol TEN_50-2411:TEN_50-2411
- added PS3: TEN_50-2412, TEN_50-2411:TEN50_TRP, symbol TEN_50-2411:TEN_50-2411
- added U1: TSR1-2450E, Converter_DCDC:Converter_DCDC_TRACO_TSR1-xxxxE_THT, symbol Regulator_Switching:TSR1-2450E
Connections:
- net +12V: now also PS3.4 (+VOUT)
- net +24V: now also PS2.1 (+VIN(VCC)), PS3.1 (+VIN(VCC)), U1.1 (Vin)
- net +5VP: now also PS2.4 (+VOUT); no longer PS1.4 (+VOUT)
- net GND: now also PS2.2 (-VIN(GND)), PS2.5 (-VOUT), PS3.2 (-VIN(GND)), PS3.5 (-VOUT), U1.2 (GND)
- net +5V renamed +5VLL
- new net +5VL: U1.3 (Vout)
- new net +5VSM: PS1.4 (+VOUT)
- no-connect marks 2 -> 6
Other:
- added sheet Connecteur (connecteurs.kicad_sch)
- added sheet led temoins (untitled.kicad_sch)
- note added: "fusible relais convertisseur:(datasheet conso ampérage) 5 VL 5 VP 12 p"
- note removed: "fusible bau +led relais led témoins changer ventilo gros condo ou bien placé :)) convertisseur:(datasheet conso ampérage) 5 VL 5 VP 12 p"
- moved on the sheet: Batcon1, Bau.1, D1, K1, PS1, U4, U6
